Commit message: Test Kuka and Vispa motion planning

File: test/data/eu-rise/eurise_scene.urdf (robot description, URDF)
Before this commit: robot Spacecraft, 256 links, 255 joints
Links:
- link CC_link: geometry visual mesh filename=./meshes/v_cargo_compartment.dae
- link IIWA14_LINK_0_link: geometry collision mesh filename=./meshes/v_kuka_link_0.dae; visual mesh filename=./meshes/v_kuka_link_0.dae
- link IIWA14_LINK_1_link: geometry collision mesh filename=./meshes/v_kuka_link_1.dae; visual mesh filename=./meshes/v_kuka_link_1.dae
- link IIWA14_LINK_2_link: geometry collision mesh filename=./meshes/v_kuka_link_2.dae; visual mesh filename=./meshes/v_kuka_link_2.dae
- link IIWA14_LINK_3_link: geometry collision mesh filename=./meshes/v_kuka_link_3.dae; visual mesh filename=./meshes/v_kuka_link_3.dae
- link IIWA14_LINK_4_link: geometry collision mesh filename=./meshes/v_kuka_link_4.dae; visual mesh filename=./meshes/v_kuka_link_4.dae
- link IIWA14_LINK_5_link: geometry collision mesh filename=./meshes/v_kuka_link_5.dae; visual mesh filename=./meshes/v_kuka_link_5.dae
- link IIWA14_LINK_6_link: geometry collision mesh filename=./meshes/v_kuka_link_6.dae; visual mesh filename=./meshes/v_kuka_link_6.dae
- link IIWA14_LINK_7_link: geometry collision box size=0.15 0.15 0.15; visual mesh filename=./meshes/v_kuka_link_7-MF-Touch-pneumatisch.dae
- link VISPA_LINK_0_link: geometry collision mesh filename=./meshes/b_vispa_link_0.dae; visual mesh filename=./meshes/v_vispa_link_0.dae
- link VISPA_LINK_1_link: geometry collision mesh filename=./meshes/b_vispa_link_1.dae; visual mesh filename=./meshes/v_vispa_link_1.dae
- link VISPA_LINK_2_link: geometry collision mesh filename=./meshes/b_vispa_link_2.dae; visual mesh filename=./meshes/v_vispa_link_2.dae
- link VISPA_LINK_3_link: geometry collision mesh filename=./meshes/b_vispa_link_3.dae; visual mesh filename=./meshes/v_vispa_link_3.dae
- link VISPA_LINK_4_link: geometry collision mesh filename=./meshes/b_vispa_link_4.dae; visual mesh filename=./meshes/v_vispa_link_4.dae
- link VISPA_LINK_5_link: geometry collision cylinder length=0.3 radius=0.085; visual mesh filename=./meshes/v_vispa_link_5.dae
- link VISPA_LINK_6_link: geometry collision mesh filename=./meshes/b_vispa_link_6.dae; visual mesh filename=./meshes/v_vispa_link_6.dae
- link WALLS_link: geometry collision mesh filename=./meshes/b_walls.dae; visual mesh filename=./meshes/b_walls.dae

Commit message: Test motion planning for kuka

File: test/data/eu-rise/eurise_scene.urdf (robot description, URDF)
Before this commit: robot Spacecraft, 256 links, 255 joints
Links:
- link IIWA14_LINK_7_link: geometry collision mesh filename=./meshes/v_kuka_link_7-MF-Touch-pneumatisch.dae; visual mesh filename=./meshes/v_kuka_link_7-MF-Touch-pneumatisch.dae
